File: mm_power.kicad_sch (KiCad schematic)
At the start: 1 part, among them J5 Conn_01x02

Commit message: fin tp2
Parts:
- added C7, C8: 1uF, symbol Device:C
- added U2: LP5907MFX-1.2, Package_TO_SOT_SMD:SOT-23-5, symbol Regulator_Linear:LP5907MFX-1.2
Connections:
- net GND: now also C7.2, C8.2, U2.2 (GND)
- new net: C7.1, U2.1 (IN), U2.3 (EN)
- new net: C8.1, U2.5 (OUT)
Changed lines of the file:
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@@
   (junction (at 86.36 82.55) (diameter 0) (color 0 0 0 0)
   )
+  (junction (at 137.16 48.26) (diameter 0) (color 0 0 0 0)
+  )
+  (junction (at 147.32 62.23) (diameter 0) (color 0 0 0 0)
+  )
   (junction (at 86.36 95.25) (diameter 0) (color 0 0 0 0)
   )
+  (junction (at 132.08 48.26) (diameter 0) (color 0 0 0 0)
+  )
+  (wire (pts (xy 147.32 58.42) (xy 147.32 62.23))
+    (stroke (width 0) (type default))
+  )
   (wire (pts (xy 86.36 90.17) (xy 86.36 95.25))
     (stroke (width 0) (type default))
   )
+  (wire (pts (xy 162.56 59.69) (xy 162.56 62.23))
+    (stroke (width 0) (type default))
+  )
+  (wire (pts (xy 137.16 48.26) (xy 139.7 48.26))
+    (stroke (width 0) (type default))
+  )
   (wire (pts (xy 95.25 82.55) (xy 86.36 82.55))
     (stroke (width 0) (type default))
@@
     (stroke (width 0) (type default))
   )
+  (wire (pts (xy 154.94 48.26) (xy 162.56 48.26))
+    (stroke (width 0) (type default))
+  )
   (wire (pts (xy 95.25 92.71) (xy 95.25 95.25))
     (stroke (width 0) (type default))
   )
+  (wire (pts (xy 132.08 44.45) (xy 86.36 44.45))
+    (stroke (width 0) (type default))
+  )
+  (wire (pts (xy 137.16 50.8) (xy 137.16 48.26))
+    (stroke (width 0) (type default))
+  )
+  (wire (pts (xy 132.08 48.26) (xy 137.16 48.26))
+    (stroke (width 0) (type default))
+  )
   (wire (pts (xy 80.01 87.63) (xy 86.36 87.63))
     (stroke (width 0) (type default))
   )
+  (wire (pts (xy 162.56 62.23) (xy 147.32 62.23))
+    (stroke (width 0) (type default))
+  )
+  (wire (pts (xy 132.08 44.45) (xy 132.08 48.26))
+    (stroke (width 0) (type default))
+  )
+  (wire (pts (xy 147.32 62.23) (xy 147.32 66.04))
+    (stroke (width 0) (type default))
+  )
+  (wire (pts (xy 139.7 50.8) (xy 137.16 50.8))
+    (stroke (width 0) (type default))
+  )
   (wire (pts (xy 86.36 95.25) (xy 86.36 100.33))
     (stroke (width 0) (type default))
@@
     (stroke (width 0) (type default))
   )
+  (wire (pts (xy 132.08 48.26) (xy 132.08 52.07))
+    (stroke (width 0) (type default))
+  )
   (wire (pts (xy 86.36 82.55) (xy 86.36 87.63))
     (stroke (width 0) (type default))
   )
+  (wire (pts (xy 86.36 44.45) (xy 86.36 72.39))
+    (stroke (width 0) (type default))
+  )
+  (wire (pts (xy 132.08 62.23) (xy 147.32 62.23))
+    (stroke (width 0) (type default))
+  )
+  (wire (pts (xy 162.56 48.26) (xy 162.56 52.07))
+    (stroke (width 0) (type default))
+  )
+  (wire (pts (xy 132.08 59.69) (xy 132.08 62.23))
+    (stroke (width 0) (type default))
+  )
   (wire (pts (xy 80.01 90.17) (xy 86.36 90.17))
     (stroke (width 0) (type default))
   )
   (symbol (lib_id "power:+BATT") (at 86.36 74.93 0) (unit 1)
-    (in_bom yes) (on_board yes) (dnp no) (fields_autoplaced)
+    (in_bom yes) (on_board yes) (dnp no)
     (property "Reference" "#PWR036" (at 86.36 78.74 0)
       (effects (font (size 1.27 1.27)) hide)
@@
         (path "/d8fa4cba-2469-4231-847f-065b6b829f44/3f9b0845-5778-418c-a7a8-03da2392145e"
           (reference "#PWR036") (unit 1)
+        )
+      )
+    )
+  )
+  (symbol (lib_id "Regulator_Linear:LP5907MFX-1.2") (at 147.32 50.8 0) (unit 1)
+    (in_bom yes) (on_board yes) (dnp no) (fields_autoplaced)
+    (property "Reference" "U2" (at 147.32 40.64 0)
+      (effects (font (size 1.27 1.27)))
+    )
+    (property "Value" "LP5907MFX-1.2" (at 147.32 43.18 0)
+      (effects (font (size 1.27 1.27)))
+    )
+    (property "Footprint" "Package_TO_SOT_SMD:SOT-23-5" (at 147.32 41.91 0)
+      (effects (font (size 1.27 1.27)) hide)
+    )
+    (property "Datasheet" "http://www.ti.com/lit/ds/symlink/lp5907.pdf" (at 147.32 38.1 0)
+      (effects (font (size 1.27 1.27)) hide)
+    )
+    (pin "1")
+    (pin "5")
+    (pin "3")
+    (pin "4")
+    (pin "2")
+    (instances
+      (project "minimouse"
+        (path "/d8fa4cba-2469-4231-847f-065b6b829f44/3f9b0845-5778-418c-a7a8-03da2392145e"
+          (reference "U2") (unit 1)
         )
       )
@@
     )
   )
+  (symbol (lib_id "Device:C") (at 162.56 55.88 0) (unit 1)
+    (in_bom yes) (on_board yes) (dnp no) (fields_autoplaced)
+    (property "Reference" "C8" (at 166.37 54.61 0)
+      (effects (font (size 1.27 1.27)) (justify left))
+    )
+    (property "Value" "1uF" (at 166.37 57.15 0)
+      (effects (font (size 1.27 1.27)) (justify left))
+    )
+    (property "Footprint" "" (at 163.5252 59.69 0)
+      (effects (font (size 1.27 1.27)) hide)
+    )
+    (property "Datasheet" "~" (at 162.56 55.88 0)
+      (effects (font (size 1.27 1.27)) hide)
+    )
+    (pin "2")
+    (pin "1")
+    (instances
+      (project "minimouse"
+        (path "/d8fa4cba-2469-4231-847f-065b6b829f44/3f9b0845-5778-418c-a7a8-03da2392145e"
+          (reference "C8") (unit 1)
+        )
+      )
+    )
+  )
+  (symbol (lib_id "Device:C") (at 132.08 55.88 0) (unit 1)
+    (in_bom yes) (on_board yes) (dnp no) (fields_autoplaced)
+    (property "Reference" "C7" (at 135.89 54.61 0)
+      (effects (font (size 1.27 1.27)) (justify left))
+    )
+    (property "Value" "1uF" (at 135.89 57.15 0)
+      (effects (font (size 1.27 1.27)) (justify left))
+    )
+    (property "Footprint" "" (at 133.0452 59.69 0)
+      (effects (font (size 1.27 1.27)) hide)
+    )
+    (property "Datasheet" "~" (at 132.08 55.88 0)
+      (effects (font (size 1.27 1.27)) hide)
+    )
+    (pin "2")
+    (pin "1")
+    (instances
+      (project "minimouse"
+        (path "/d8fa4cba-2469-4231-847f-065b6b829f44/3f9b0845-5778-418c-a7a8-03da2392145e"
+          (reference "C7") (unit 1)
+        )
+      )
+    )
+  )
   (symbol (lib_id "Connector_Generic:Conn_01x02") (at 74.93 90.17 180) (unit 1)
     (in_bom yes) (on_board yes) (dnp no) (fields_autoplaced)
@@
         )
       )
+    )
+  )
+  (symbol (lib_id "power:GND") (at 147.32 66.04 0) (unit 1)
+    (in_bom yes) (on_board yes) (dnp no) (fields_autoplaced)
+    (property "Reference" "#PWR08" (at 147.32 72.39 0)
+      (effects (font (size 1.27 1.27)) hide)
+    )
+    (property "Value" "GND" (at 147.32 71.12 0)
+      (effects (font (size 1.27 1.27)))
+    )
+    (property "Footprint" "" (at 147.32 66.04 0)
+      (effects (font (size 1.27 1.27)) hide)
+    )
+    (property "Datasheet" "" (at 147.32 66.04 0)
+      (effects (font (size 1.27 1.27)) hide)
+    )
+    (pin "1")
+    (instances
+      (project "minimouse"
+        (path "/d8fa4cba-2469-4231-847f-065b6b829f44/3f9b0845-5778-418c-a7a8-03da2392145e"
+          (reference "#PWR08") (unit 1)
+        )
+      )

Commit message: TP2
Parts:
- added D1: LED, LED_SMD:LED_0603_1608Metric, symbol Device:LED
- added R13: R, Resistor_SMD:R_0603_1608Metric, symbol Device:R
- C7, C8: footprint (none) -> Capacitor_SMD:C_0603_1608Metric
Connections:
- net GND: now also D1.1 (K)
- net +3.3V: now reaches C8.1, U2.5 (OUT)
- net +3.3V: now also R13.1
- new net: D1.2 (A), R13.2
Changed lines of the file:
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@@
   (junction (at 132.08 48.26) (diameter 0) (color 0 0 0 0)
   )
+  (junction (at 162.56 48.26) (diameter 0) (color 0 0 0 0)
+  )
   (wire (pts (xy 147.32 58.42) (xy 147.32 62.23))
     (stroke (width 0) (type default))
@@
     (stroke (width 0) (type default))
   )
+  (wire (pts (xy 208.28 73.66) (xy 208.28 83.82))
+    (stroke (width 0) (type default))
+  )
   (wire (pts (xy 95.25 82.55) (xy 86.36 82.55))
     (stroke (width 0) (type default))
@@
     (stroke (width 0) (type default))
   )
+  (wire (pts (xy 162.56 48.26) (xy 208.28 48.26))
+    (stroke (width 0) (type default))
+  )
   (wire (pts (xy 95.25 92.71) (xy 95.25 95.25))
     (stroke (width 0) (type default))
@@
     (stroke (width 0) (type default))
   )
+  (wire (pts (xy 162.56 43.18) (xy 162.56 48.26))
+    (stroke (width 0) (type default))
+  )
   (wire (pts (xy 147.32 62.23) (xy 147.32 66.04))
     (stroke (width 0) (type default))
@@
     (stroke (width 0) (type default))
   )
+  (wire (pts (xy 208.28 58.42) (xy 208.28 66.04))
+    (stroke (width 0) (type default))
+  )
   (wire (pts (xy 95.25 95.25) (xy 86.36 95.25))
+    (stroke (width 0) (type default))
+  )
+  (wire (pts (xy 208.28 48.26) (xy 208.28 50.8))
     (stroke (width 0) (type default))
   )
@@
         (path "/d8fa4cba-2469-4231-847f-065b6b829f44/3f9b0845-5778-418c-a7a8-03da2392145e"
           (reference "#PWR036") (unit 1)
+        )
+      )
+    )
+  )
+  (symbol (lib_id "power:+3.3V") (at 162.56 43.18 0) (unit 1)
+    (in_bom yes) (on_board yes) (dnp no) (fields_autoplaced)
+    (property "Reference" "#PWR015" (at 162.56 46.99 0)
+      (effects (font (size 1.27 1.27)) hide)
+    )
+    (property "Value" "+3.3V" (at 162.56 38.1 0)
+      (effects (font (size 1.27 1.27)))
+    )
+    (property "Footprint" "" (at 162.56 43.18 0)
+      (effects (font (size 1.27 1.27)) hide)
+    )
+    (property "Datasheet" "" (at 162.56 43.18 0)
+      (effects (font (size 1.27 1.27)) hide)
+    )
+    (pin "1")
+    (instances
+      (project "minimouse"
+        (path "/d8fa4cba-2469-4231-847f-065b6b829f44/3f9b0845-5778-418c-a7a8-03da2392145e"
+          (reference "#PWR015") (unit 1)
         )
       )
@@
     )
   )
+  (symbol (lib_id "power:GND") (at 208.28 83.82 0) (unit 1)
+    (in_bom yes) (on_board yes) (dnp no) (fields_autoplaced)
+    (property "Reference" "#PWR014" (at 208.28 90.17 0)
+      (effects (font (size 1.27 1.27)) hide)
+    )
+    (property "Value" "GND" (at 208.28 88.9 0)
+      (effects (font (size 1.27 1.27)))
+    )
+    (property "Footprint" "" (at 208.28 83.82 0)
+      (effects (font (size 1.27 1.27)) hide)
+    )
+    (property "Datasheet" "" (at 208.28 83.82 0)
+      (effects (font (size 1.27 1.27)) hide)
+    )
+    (pin "1")
+    (instances
+      (project "minimouse"
+        (path "/d8fa4cba-2469-4231-847f-065b6b829f44/3f9b0845-5778-418c-a7a8-03da2392145e"
+          (reference "#PWR014") (unit 1)
+        )
+      )
+    )
+  )
+  (symbol (lib_id "Device:R") (at 208.28 54.61 0) (unit 1)
+    (in_bom yes) (on_board yes) (dnp no) (fields_autoplaced)
+    (property "Reference" "R13" (at 210.82 53.34 0)
+      (effects (font (size 1.27 1.27)) (justify left))
+    )
+    (property "Value" "R" (at 210.82 55.88 0)
+      (effects (font (size 1.27 1.27)) (justify left))
+    )
+    (property "Footprint" "Resistor_SMD:R_0603_1608Metric" (at 206.502 54.61 90)
+      (effects (font (size 1.27 1.27)) hide)
+    )
+    (property "Datasheet" "~" (at 208.28 54.61 0)
+      (effects (font (size 1.27 1.27)) hide)
+    )
+    (pin "2")
+    (pin "1")
+    (instances
+      (project "minimouse"
+        (path "/d8fa4cba-2469-4231-847f-065b6b829f44/3f9b0845-5778-418c-a7a8-03da2392145e"
+          (reference "R13") (unit 1)
+        )
+      )
+    )
+  )
+  (symbol (lib_id "Device:LED") (at 208.28 69.85 90) (unit 1)
+    (in_bom yes) (on_board yes) (dnp no) (fields_autoplaced)
+    (property "Reference" "D1" (at 212.09 70.1675 90)
+      (effects (font (size 1.27 1.27)) (justify right))
+    )
+    (property "Value" "LED" (at 212.09 72.7075 90)
+      (effects (font (size 1.27 1.27)) (justify right))
+    )
+    (property "Footprint" "LED_SMD:LED_0603_1608Metric" (at 208.28 69.85 0)
+      (effects (font (size 1.27 1.27)) hide)
+    )
+    (property "Datasheet" "~" (at 208.28 69.85 0)
+      (effects (font (size 1.27 1.27)) hide)
+    )
+    (pin "2")
+    (pin "1")
+    (instances
+      (project "minimouse"
+        (path "/d8fa4cba-2469-4231-847f-065b6b829f44/3f9b0845-5778-418c-a7a8-03da2392145e"
+          (reference "D1") (unit 1)
+        )
+      )
+    )
+  )
   (symbol (lib_id "Device:C") (at 162.56 55.88 0) (unit 1)
     (in_bom yes) (on_board yes) (dnp no) (fields_autoplaced)
@@
       (effects (font (size 1.27 1.27)) (justify left))
     )
-    (property "Footprint" "" (at 163.5252 59.69 0)
+    (property "Footprint" "Capacitor_SMD:C_0603_1608Metric" (at 163.5252 59.69 0)
       (effects (font (size 1.27 1.27)) hide)
     )
@@
       (effects (font (size 1.27 1.27)) (justify left))
     )
-    (property "Footprint" "" (at 133.0452 59.69 0)
-      (effects (font (size 1.27 1.27)) hide)
-    )
+    (property "Footprint" "Capacitor_SMD:C_0603_1608Metric" (at 133.0452 59.69 0)
+      (effects (font (size 1.27 1.27)) hide)
+    )
