File: mm_motor_control.kicad_sch (KiCad schematic)
At the start: 0 parts

Commit message: fin tp2
Parts:
- added C9: C, symbol Device:C
- added CEN: 10nF, symbol Device:C
- added CRCOFF: 22nF, symbol Device:C
- added CSPOL: 22uF, symbol Device:C
- added Cs: 2.2uF, symbol Device:C
- added R10, R11: 10K, symbol Device:R
- added R12: R, symbol Device:R
- added REN: 18K, symbol Device:R
- added ROFF: 47K, symbol Device:R
- added RRCOFF: 1K, symbol Device:R
- added RSNSA: 330 m, symbol Device:R
- added RSNSB: 330m, symbol Device:R
- added U3: STSPIN240, Package_DFN_QFN:VQFN-16-1EP_3x3mm_P0.5mm_EP1.8x1.8mm, symbol Driver_Motor:STSPIN240
Connections:
- net EN: now also REN.1
- net FAULT: now also U3.13 (EN/FLT)
- net OUT_A1: now also RSNSA.1, U3.3 (OUTA1), U3.4 (SENSEA), U3.5 (OUTA2)
- net OUT_B1: now also RSNSB.1, U3.10 (OUTB1), U3.8 (OUTB2), U3.9 (SENSEB)
- net PHASE_A: now also U3.1 (PHA), U3.2 (PWMA)
- net PHASE_B: now also U3.15 (PHB)
- net PWM_B: now also U3.16 (PWMB)
- net STBY/RESET: now also C9.1, R12.2, U3.14 (STBY/RESET)
- new net: CEN.1, REN.2
- new net: CSPOL.2, Cs.2
- new net: ROFF.1, RRCOFF.1, U3.12 (TOFF)
- new net: R10.2, R11.1, U3.11 (REF)
- new net: CRCOFF.1, RRCOFF.2
- new net +BATT: R10.1
- new net GND: C9.2, CEN.2, CRCOFF.2, R11.2, ROFF.2, RSNSA.2, RSNSB.2, U3.17 (EPAD), U3.7 (GND)
- new net VDD: R12.1
- new net VS: CSPOL.1, Cs.1, U3.6 (VS)

Commit message: TP2
Parts:
- C9: footprint (none) -> Capacitor_SMD:C_0603_1608Metric
- CEN1: renamed from CEN; footprint (none) -> Capacitor_SMD:C_0603_1608Metric
- CRCOFF1: renamed from CRCOFF; footprint (none) -> Capacitor_SMD:C_0603_1608Metric
- CSPOL1: renamed from CSPOL; footprint (none) -> Capacitor_SMD:C_0603_1608Metric
- Cs1: renamed from Cs; footprint (none) -> Capacitor_SMD:C_0603_1608Metric
- R10, R11, R12: footprint (none) -> Resistor_SMD:R_0603_1608Metric
- REN1: renamed from REN; footprint (none) -> Resistor_SMD:R_0603_1608Metric
- ROFF1: renamed from ROFF; footprint (none) -> Resistor_SMD:R_0603_1608Metric
- RRCOFF1: renamed from RRCOFF; footprint (none) -> Resistor_SMD:R_0603_1608Metric
- RSNSA1: renamed from RSNSA; footprint (none) -> Resistor_SMD:R_2512_6332Metric
- RSNSB1: renamed from RSNSB; footprint (none) -> Resistor_SMD:R_2512_6332Metric
Changed lines of the file:
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@@
   (symbol (lib_id "power:+BATT") (at 71.12 106.68 0) (unit 1)
     (in_bom yes) (on_board yes) (dnp no)
-    (property "Reference" "#PWR036" (at 71.12 110.49 0)
+    (property "Reference" "#PWR011" (at 71.12 110.49 0)
       (effects (font (size 1.27 1.27)) hide)
     )
@@
     (instances
       (project "minimouse"
-        (path "/d8fa4cba-2469-4231-847f-065b6b829f44/3f9b0845-5778-418c-a7a8-03da2392145e"
-          (reference "#PWR036") (unit 1)
-        )
         (path "/d8fa4cba-2469-4231-847f-065b6b829f44/0999fad3-9a14-4ede-b729-a71c3dbbdf8e"
           (reference "#PWR011") (unit 1)
@@
   (symbol (lib_id "Device:R") (at 148.59 88.9 0) (unit 1)
     (in_bom yes) (on_board yes) (dnp no) (fields_autoplaced)
-    (property "Reference" "RSNSA" (at 151.13 87.63 0)
+    (property "Reference" "RSNSA1" (at 151.13 87.63 0)
       (effects (font (size 1.27 1.27)) (justify left))
     )
@@
       (effects (font (size 1.27 1.27)) (justify left))
     )
-    (property "Footprint" "" (at 146.812 88.9 90)
+    (property "Footprint" "Resistor_SMD:R_2512_6332Metric" (at 146.812 88.9 90)
       (effects (font (size 1.27 1.27)) hide)
     )
@@
       (project "minimouse"
         (path "/d8fa4cba-2469-4231-847f-065b6b829f44/0999fad3-9a14-4ede-b729-a71c3dbbdf8e"
-          (reference "RSNSA") (unit 1)
+          (reference "RSNSA1") (unit 1)
         )
       )
@@
   (symbol (lib_id "Device:C") (at 63.5 107.95 0) (unit 1)
     (in_bom yes) (on_board yes) (dnp no) (fields_autoplaced)
-    (property "Reference" "CEN" (at 67.31 106.68 0)
+    (property "Reference" "CEN1" (at 67.31 106.68 0)
       (effects (font (size 1.27 1.27)) (justify left))
     )
@@
       (effects (font (size 1.27 1.27)) (justify left))
     )
-    (property "Footprint" "" (at 64.4652 111.76 0)
+    (property "Footprint" "Capacitor_SMD:C_0603_1608Metric" (at 64.4652 111.76 0)
       (effects (font (size 1.27 1.27)) hide)
     )
@@
       (project "minimouse"
         (path "/d8fa4cba-2469-4231-847f-065b6b829f44/0999fad3-9a14-4ede-b729-a71c3dbbdf8e"
-          (reference "CEN") (unit 1)
+          (reference "CEN1") (unit 1)
         )
       )
@@
   (symbol (lib_id "Device:R") (at 154.94 102.87 0) (unit 1)
     (in_bom yes) (on_board yes) (dnp no) (fields_autoplaced)
-    (property "Reference" "RSNSB" (at 157.48 101.6 0)
+    (property "Reference" "RSNSB1" (at 157.48 101.6 0)
       (effects (font (size 1.27 1.27)) (justify left))
     )
@@
       (effects (font (size 1.27 1.27)) (justify left))
     )
-    (property "Footprint" "" (at 153.162 102.87 90)
+    (property "Footprint" "Resistor_SMD:R_2512_6332Metric" (at 153.162 102.87 90)
       (effects (font (size 1.27 1.27)) hide)
     )
@@
       (project "minimouse"
         (path "/d8fa4cba-2469-4231-847f-065b6b829f44/0999fad3-9a14-4ede-b729-a71c3dbbdf8e"
-          (reference "RSNSB") (unit 1)
+          (reference "RSNSB1") (unit 1)
         )
       )
@@
       (effects (font (size 1.27 1.27)) (justify left))
     )
-    (property "Footprint" "" (at 42.8752 142.24 0)
+    (property "Footprint" "Capacitor_SMD:C_0603_1608Metric" (at 42.8752 142.24 0)
       (effects (font (size 1.27 1.27)) hide)
     )
@@
   (symbol (lib_id "Device:R") (at 50.8 97.79 90) (unit 1)
     (in_bom yes) (on_board yes) (dnp no) (fields_autoplaced)
-    (property "Reference" "REN" (at 50.8 91.44 90)
+    (property "Reference" "REN1" (at 50.8 91.44 90)
       (effects (font (size 1.27 1.27)))
     )
@@
       (effects (font (size 1.27 1.27)))
     )
-    (property "Footprint" "" (at 50.8 99.568 90)
+    (property "Footprint" "Resistor_SMD:R_0603_1608Metric" (at 50.8 99.568 90)
       (effects (font (size 1.27 1.27)) hide)
     )
@@
       (project "minimouse"
         (path "/d8fa4cba-2469-4231-847f-065b6b829f44/0999fad3-9a14-4ede-b729-a71c3dbbdf8e"
-          (reference "REN") (unit 1)
+          (reference "REN1") (unit 1)
         )
       )
@@
   (symbol (lib_id "Device:C") (at 219.71 74.93 0) (unit 1)
     (in_bom yes) (on_board yes) (dnp no) (fields_autoplaced)
-    (property "Reference" "Cs" (at 223.52 73.66 0)
+    (property "Reference" "Cs1" (at 223.52 73.66 0)
       (effects (font (size 1.27 1.27)) (justify left))
     )
@@
       (effects (font (size 1.27 1.27)) (justify left))
     )
-    (property "Footprint" "" (at 220.6752 78.74 0)
+    (property "Footprint" "Capacitor_SMD:C_0603_1608Metric" (at 220.6752 78.74 0)
       (effects (font (size 1.27 1.27)) hide)
     )
@@
       (project "minimouse"
         (path "/d8fa4cba-2469-4231-847f-065b6b829f44/0999fad3-9a14-4ede-b729-a71c3dbbdf8e"
-          (reference "Cs") (unit 1)
+          (reference "Cs1") (unit 1)
         )
       )
@@
   (symbol (lib_id "Device:C") (at 237.49 74.93 0) (unit 1)
     (in_bom yes) (on_board yes) (dnp no) (fields_autoplaced)
-    (property "Reference" "CSPOL" (at 241.3 73.66 0)
+    (property "Reference" "CSPOL1" (at 241.3 73.66 0)
       (effects (font (size 1.27 1.27)) (justify left))
     )
@@
       (effects (font (size 1.27 1.27)) (justify left))
     )
-    (property "Footprint" "" (at 238.4552 78.74 0)
+    (property "Footprint" "Capacitor_SMD:C_0603_1608Metric" (at 238.4552 78.74 0)
       (effects (font (size 1.27 1.27)) hide)
     )
@@
       (project "minimouse"
         (path "/d8fa4cba-2469-4231-847f-065b6b829f44/0999fad3-9a14-4ede-b729-a71c3dbbdf8e"
-          (reference "CSPOL") (unit 1)
+          (reference "CSPOL1") (unit 1)
         )
       )
@@
       (effects (font (size 1.27 1.27)) (justify left))
     )
-    (property "Footprint" "" (at 40.132 127 90)
+    (property "Footprint" "Resistor_SMD:R_0603_1608Metric" (at 40.132 127 90)
       (effects (font (size 1.27 1.27)) hide)
     )
@@
   (symbol (lib_id "Device:R") (at 107.95 121.92 0) (unit 1)
     (in_bom yes) (on_board yes) (dnp no) (fields_autoplaced)
-    (property "Reference" "ROFF" (at 110.49 120.65 0)
+    (property "Reference" "ROFF1" (at 110.49 120.65 0)
       (effects (font (size 1.27 1.27)) (justify left))
     )
@@
       (effects (font (size 1.27 1.27)) (justify left))
     )
-    (property "Footprint" "" (at 106.172 121.92 90)
+    (property "Footprint" "Resistor_SMD:R_0603_1608Metric" (at 106.172 121.92 90)
       (effects (font (size 1.27 1.27)) hide)
     )
@@
       (project "minimouse"
         (path "/d8fa4cba-2469-4231-847f-065b6b829f44/0999fad3-9a14-4ede-b729-a71c3dbbdf8e"
-          (reference "ROFF") (unit 1)
+          (reference "ROFF1") (unit 1)
         )
       )
@@
   (symbol (lib_id "Device:C") (at 97.79 127 0) (unit 1)
     (in_bom yes) (on_board yes) (dnp no) (fields_autoplaced)
-    (property "Reference" "CRCOFF" (at 101.6 125.73 0)
+    (property "Reference" "CRCOFF1" (at 101.6 125.73 0)
       (effects (font (size 1.27 1.27)) (justify left))
     )
@@
       (effects (font (size 1.27 1.27)) (justify left))
     )
-    (property "Footprint" "" (at 98.7552 130.81 0)
+    (property "Footprint" "Capacitor_SMD:C_0603_1608Metric" (at 98.7552 130.81 0)
       (effects (font (size 1.27 1.27)) hide)
     )
@@
       (project "minimouse"
         (path "/d8fa4cba-2469-4231-847f-065b6b829f44/0999fad3-9a14-4ede-b729-a71c3dbbdf8e"
-          (reference "CRCOFF") (unit 1)
+          (reference "CRCOFF1") (unit 1)
         )
       )
@@
   (symbol (lib_id "Device:R") (at 97.79 114.3 0) (unit 1)
     (in_bom yes) (on_board yes) (dnp no) (fields_autoplaced)
-    (property "Reference" "RRCOFF" (at 100.33 113.03 0)
+    (property "Reference" "RRCOFF1" (at 100.33 113.03 0)
       (effects (font (size 1.27 1.27)) (justify left))
     )
@@
       (effects (font (size 1.27 1.27)) (justify left))
     )
-    (property "Footprint" "" (at 96.012 114.3 90)
+    (property "Footprint" "Resistor_SMD:R_0603_1608Metric" (at 96.012 114.3 90)
       (effects (font (size 1.27 1.27)) hide)
     )
@@
       (project "minimouse"
         (path "/d8fa4cba-2469-4231-847f-065b6b829f44/0999fad3-9a14-4ede-b729-a71c3dbbdf8e"
-          (reference "RRCOFF") (unit 1)
+          (reference "RRCOFF1") (unit 1)
         )
       )
@@
       (effects (font (size 1.27 1.27)) (justify left))
     )
-    (property "Footprint" "" (at 75.692 118.11 90)
+    (property "Footprint" "Resistor_SMD:R_0603_1608Metric" (at 75.692 118.11 90)
       (effects (font (size 1.27 1.27)) hide)
     )
@@
       (effects (font (size 1.27 1.27)) (justify left))
     )
-    (property "Footprint" "" (at 75.692 134.62 90)
-      (effects (font (size 1.27 1.27)) hide)
-    )
+    (property "Footprint" "Resistor_SMD:R_0603_1608Metric" (at 75.692 134.62 90)
+      (effects (font (size 1.27 1.27)) hide)
+    )

Commit message: tp2p2
Changed lines of the file:
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@@
   (junction (at 138.43 83.82) (diameter 0) (color 0 0 0 0)
   )
-  (junction (at 193.04 118.11) (diameter 0) (color 0 0 0 0)
-  )
   (junction (at 41.91 133.35) (diameter 0) (color 0 0 0 0)
   )
@@
     (stroke (width 0) (type default))
   )
-  (wire (pts (xy 193.04 118.11) (xy 229.87 118.11))
-    (stroke (width 0) (type default))
-  )
